File: kicad-cnc/CNC.kicad_pcb (KiCad board)
At the start: 4 copper layers, 90 x 70 mm, 14 parts, among them J1 Conn_02x25_Odd_Even, J2 Conn_02x08_Odd_Even, J3 Conn_01x04, U1 74AHC595, U2 ESP32_DevKitC_V4, U3 74AHC595

Commit message: started with the base pcb
Connections:
- J1 pad 25: LIMIT_X1_POS -> OUT_{1}
- J1 pad 26: LIMIT_X1_NEG -> OUT_{2}
- J1 pad 27: LIMIT_X2_POS -> LIMIT_X1_POS
- J1 pad 28: LIMIT_X2_NEG -> LIMIT_X1_NEG
- J1 pad 29: LIMIT_Y_POS -> LIMIT_X2_POS
- J1 pad 30: LIMIT_Y_NEG -> LIMIT_X2_NEG
- J1 pad 31: LIMIT_Z_POS -> LIMIT_Y_POS
- J1 pad 32: LIMIT_Z_NEG -> LIMIT_Y_NEG
- J1 pad 33: PROBE -> LIMIT_Z_POS
- J1 pad 34: IN_{0} -> LIMIT_Z_NEG
- J1 pad 35: IN_{1} -> PROBE
- J1 pad 36: IN_{2} -> IN_{0}
- J1 pad 37: unconnected-(J1-Pad37) -> IN_{1}
- J1 pad 38: unconnected-(J1-Pad38) -> IN_{2}
- U3 pad 3: unconnected-(U3-Pad3) -> OUT_{1}
- U3 pad 4: unconnected-(U3-Pad4) -> OUT_{2}
Routing:
- net OUT_{2}: track 0.00 -> 29.8 mm
- net OUT_{1}: track 0.00 -> 26.7 mm
- net SD_MOSI: track 35.5 -> 16.8 mm
- net I2S_BCK: track 44.2 -> 32.3 mm, vias 0 -> 2
- net Net-(U1-Pad9): track 21.3 -> 11.4 mm, vias 0 -> 2
- net I2S_DATA: track 52.3 -> 45.3 mm, vias 0 -> 2
- net I2S_WS: track 68.2 -> 62.2 mm, vias 2 -> 5
- net LIMIT_X1_NEG: track 55.5 -> 52.3 mm
- net LIMIT_X1_POS: track 54.5 -> 51.3 mm
- net LIMIT_X2_NEG: track 52.2 -> 49.2 mm
- net LIMIT_X2_POS: track 51.2 -> 48.3 mm
- net LIMIT_Y_NEG: track 49.8 -> 47.2 mm
- net LIMIT_Y_POS: track 47.8 -> 45.3 mm
- net PROBE: track 52.5 -> 50.2 mm
- net GND: track 3.74 -> 6.03 mm, vias 74 -> 75
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