File: kicad-cnc-connectors/kicad-cnc-connectors.kicad_pcb (KiCad board)
At the start: 2 copper layers, 90 x 60 mm, 37 parts, among them J1 Conn_01x03, J10 Conn_01x06, J11 Conn_01x03, J12 Conn_01x03, J13 Conn_01x06, J14 Conn_01x03, J15 Conn_01x03, J16 Conn_01x03, J17 Conn_01x03, J18 Conn_01x03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

Commit message: updated PCBs
Parts:
- R1, R10, R11, R12, R2, R3, R4, R5, R6, R7, R8, R9: value R -> 10k
