File: kicad-cnc-connectors/kicad-cnc-connectors.kicad_sch (KiCad schematic)
At the start: 37 parts, among them J1 Conn_01x03, J10 Conn_01x06, J11 Conn_01x03, J12 Conn_01x03, J13 Conn_01x06, J14 Conn_01x03, J15 Conn_01x03, J16 Conn_01x03, J17 Conn_01x03, J18 Conn_01x03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

Commit message: updated PCBs
Parts:
- R1, R10, R11, R12, R2, R3, R4, R5, R6, R7, R8, R9: value R -> 10k
Changed lines of the file:
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@@
     (in_bom yes) (on_board yes)
     (property "Reference" "R1" (id 0) (at 43.18 101.6 90))
-    (property "Value" "R" (id 1) (at 46.99 101.6 90))
+    (property "Value" "10k" (id 1) (at 46.99 101.6 90))
     (property "Footprint" "Resistor_SMD:R_0402_1005Metric" (id 2) (at 45.72 105.918 90)
       (effects (font (size 1.27 1.27)) hide)
@@
     (in_bom yes) (on_board yes)
     (property "Reference" "R8" (id 0) (at 43.18 137.16 90))
-    (property "Value" "R" (id 1) (at 46.99 137.16 90))
+    (property "Value" "10k" (id 1) (at 46.99 137.16 90))
     (property "Footprint" "Resistor_SMD:R_0402_1005Metric" (id 2) (at 45.72 141.478 90)
       (effects (font (size 1.27 1.27)) hide)
@@
     (in_bom yes) (on_board yes)
     (property "Reference" "R7" (id 0) (at 43.18 132.08 90))
-    (property "Value" "R" (id 1) (at 46.99 132.08 90))
+    (property "Value" "10k" (id 1) (at 46.99 132.08 90))
     (property "Footprint" "Resistor_SMD:R_0402_1005Metric" (id 2) (at 45.72 136.398 90)
       (effects (font (size 1.27 1.27)) hide)
@@
     (in_bom yes) (on_board yes)
     (property "Reference" "R3" (id 0) (at 43.18 111.76 90))
-    (property "Value" "R" (id 1) (at 46.99 111.76 90))
+    (property "Value" "10k" (id 1) (at 46.99 111.76 90))
     (property "Footprint" "Resistor_SMD:R_0402_1005Metric" (id 2) (at 45.72 116.078 90)
       (effects (font (size 1.27 1.27)) hide)
@@
     (in_bom yes) (on_board yes)
     (property "Reference" "R6" (id 0) (at 43.18 127 90))
-    (property "Value" "R" (id 1) (at 46.99 127 90))
+    (property "Value" "10k" (id 1) (at 46.99 127 90))
     (property "Footprint" "Resistor_SMD:R_0402_1005Metric" (id 2) (at 45.72 131.318 90)
       (effects (font (size 1.27 1.27)) hide)
@@
     (in_bom yes) (on_board yes)
     (property "Reference" "R12" (id 0) (at 43.18 157.48 90))
-    (property "Value" "R" (id 1) (at 46.99 157.48 90))
+    (property "Value" "10k" (id 1) (at 46.99 157.48 90))
     (property "Footprint" "Resistor_SMD:R_0402_1005Metric" (id 2) (at 45.72 161.798 90)
       (effects (font (size 1.27 1.27)) hide)
@@
     (in_bom yes) (on_board yes)
     (property "Reference" "R11" (id 0) (at 43.18 152.4 90))
-    (property "Value" "R" (id 1) (at 46.99 152.4 90))
+    (property "Value" "10k" (id 1) (at 46.99 152.4 90))
     (property "Footprint" "Resistor_SMD:R_0402_1005Metric" (id 2) (at 45.72 156.718 90)
       (effects (font (size 1.27 1.27)) hide)
@@
     (in_bom yes) (on_board yes)
     (property "Reference" "R5" (id 0) (at 43.18 121.92 90))
-    (property "Value" "R" (id 1) (at 46.99 121.92 90))
+    (property "Value" "10k" (id 1) (at 46.99 121.92 90))
     (property "Footprint" "Resistor_SMD:R_0402_1005Metric" (id 2) (at 45.72 126.238 90)
       (effects (font (size 1.27 1.27)) hide)
@@
     (in_bom yes) (on_board yes)
     (property "Reference" "R2" (id 0) (at 43.18 106.68 90))
-    (property "Value" "R" (id 1) (at 46.99 106.68 90))
+    (property "Value" "10k" (id 1) (at 46.99 106.68 90))
     (property "Footprint" "Resistor_SMD:R_0402_1005Metric" (id 2) (at 45.72 110.998 90)
       (effects (font (size 1.27 1.27)) hide)
@@
     (in_bom yes) (on_board yes)
     (property "Reference" "R4" (id 0) (at 43.18 116.84 90))
-    (property "Value" "R" (id 1) (at 46.99 116.84 90))
+    (property "Value" "10k" (id 1) (at 46.99 116.84 90))
     (property "Footprint" "Resistor_SMD:R_0402_1005Metric" (id 2) (at 45.72 121.158 90)
       (effects (font (size 1.27 1.27)) hide)
@@
     (in_bom yes) (on_board yes)
     (property "Reference" "R9" (id 0) (at 43.18 142.24 90))
-    (property "Value" "R" (id 1) (at 46.99 142.24 90))
+    (property "Value" "10k" (id 1) (at 46.99 142.24 90))
     (property "Footprint" "Resistor_SMD:R_0402_1005Metric" (id 2) (at 45.72 146.558 90)
       (effects (font (size 1.27 1.27)) hide)
@@
     (in_bom yes) (on_board yes)
     (property "Reference" "R10" (id 0) (at 43.18 147.32 90))
-    (property "Value" "R" (id 1) (at 46.99 147.32 90))
+    (property "Value" "10k" (id 1) (at 46.99 147.32 90))
     (property "Footprint" "Resistor_SMD:R_0402_1005Metric" (id 2) (at 45.72 151.638 90)
       (effects (font (size 1.27 1.27)) hide)
@@
     )
     (path "/054c4bec-9368-4d60-b030-f824f36fcae0"
-      (reference "R1") (unit 1) (value "R") (footprint "Resistor_SMD:R_0402_1005Metric")
+      (reference "R1") (unit 1) (value "10k") (footprint "Resistor_SMD:R_0402_1005Metric")
     )
     (path "/d607396f-c6f9-4abb-aca9-ae31b1a8d243"
-      (reference "R2") (unit 1) (value "R") (footprint "Resistor_SMD:R_0402_1005Metric")
+      (reference "R2") (unit 1) (value "10k") (footprint "Resistor_SMD:R_0402_1005Metric")
     )
     (path "/83d8a4ef-2acd-4bdb-87a6-716abb10a33a"
-      (reference "R3") (unit 1) (value "R") (footprint "Resistor_SMD:R_0402_1005Metric")
+      (reference "R3") (unit 1) (value "10k") (footprint "Resistor_SMD:R_0402_1005Metric")
     )
     (path "/e91c4324-5bb3-4fda-a069-e0bc61dac6bd"
-      (reference "R4") (unit 1) (value "R") (footprint "Resistor_SMD:R_0402_1005Metric")
+      (reference "R4") (unit 1) (value "10k") (footprint "Resistor_SMD:R_0402_1005Metric")
     )
     (path "/c41f6f7d-6efe-4709-9537-157117d528af"
-      (reference "R5") (unit 1) (value "R") (footprint "Resistor_SMD:R_0402_1005Metric")
+      (reference "R5") (unit 1) (value "10k") (footprint "Resistor_SMD:R_0402_1005Metric")
     )
     (path "/932f5c99-cb3e-4445-be27-9db800b1318a"
-      (reference "R6") (unit 1) (value "R") (footprint "Resistor_SMD:R_0402_1005Metric")
+      (reference "R6") (unit 1) (value "10k") (footprint "Resistor_SMD:R_0402_1005Metric")
     )
     (path "/77706280-feb8-4164-885e-d64ddc70ff3e"
-      (reference "R7") (unit 1) (value "R") (footprint "Resistor_SMD:R_0402_1005Metric")
+      (reference "R7") (unit 1) (value "10k") (footprint "Resistor_SMD:R_0402_1005Metric")
     )
     (path "/691769b5-efbe-42d0-aafd-f02d8fc786ba"
-      (reference "R8") (unit 1) (value "R") (footprint "Resistor_SMD:R_0402_1005Metric")
+      (reference "R8") (unit 1) (value "10k") (footprint "Resistor_SMD:R_0402_1005Metric")
     )
     (path "/f09a47bc-d53e-417e-86c0-43fb06ee8d6a"
-      (reference "R9") (unit 1) (value "R") (footprint "Resistor_SMD:R_0402_1005Metric")
+      (reference "R9") (unit 1) (value "10k") (footprint "Resistor_SMD:R_0402_1005Metric")
     )
     (path "/face11e6-90c9-4893-b320-ec98672b3b5d"
-      (reference "R10") (unit 1) (value "R") (footprint "Resistor_SMD:R_0402_1005Metric")
+      (reference "R10") (unit 1) (value "10k") (footprint "Resistor_SMD:R_0402_1005Metric")
     )
     (path "/c035dd50-bd95-437e-a52b-dff47f00df41"
-      (reference "R11") (unit 1) (value "R") (footprint "Resistor_SMD:R_0402_1005Metric")
+      (reference "R11") (unit 1) (value "10k") (footprint "Resistor_SMD:R_0402_1005Metric")
     )
     (path "/bcdc22b7-bacd-4458-9499-a8bcb1a8b301"
-      (reference "R12") (unit 1) (value "R") (footprint "Resistor_SMD:R_0402_1005Metric")
-    )
-  )
+      (reference "R12") (unit 1) (value "10k") (footprint "Resistor_SMD:R_0402_1005Metric")
+    )
+  )
