File: kicad-cnc-esp32/kicad-cnc-esp32.kicad_pcb (KiCad board)
At the start: 2 copper layers, 90 x 70 mm, 28 parts, among them J1 Conn_02x25_Odd_Even, J2 Conn_01x04, J3 Conn_02x08_Odd_Even, U1 SN74LVC4245A, U2 ESP32_DevKitC_V4, U3 SN74LVC4245A, U4 74AHC595, U5 74AHC595, U6 SN74LVC4245A, U7 SN74LVC4245A

Commit message: updated PCBs
Parts:
- C1, C10, C11, C12, C13, C14, C2, C3, C4, C5, C6, C7, C8, C9: value C -> 4.7uF
